Commit message: Corrected previous commit by mapping correct sensory feedback. Check init_pos and establish final joint positions and set gains. Not yet standing with init_pos.

File: coman_description/model/model.urdf (robot description, URDF)
Before this commit: robot coman, 64 links, 63 joints
Links:
- link DWL: geometry collision mesh filename=package://coman_description/model/meshes/simple/Torso1.STL scale=0.03937 0.03937 0.03937; visual mesh filename=package://coman_description/model/meshes/Torso1.STL scale=0.03937 0.03937 0.03937
- link DWS: geometry collision mesh filename=package://coman_description/model/meshes/simple/Torso2.STL scale=0.03937 0.03937 0.03937; visual mesh filename=package://coman_description/model/meshes/Torso2.STL scale=0.03937 0.03937 0.03937
- link DWYTorso: geometry collision mesh filename=package://coman_description/model/meshes/simple/Torso3.STL scale=0.03937 0.03937 0.03937; visual mesh filename=package://coman_description/model/meshes/Torso3.STL scale=0.03937 0.03937 0.03937
- link LElb: geometry collision mesh filename=package://coman_description/model/meshes/simple/Elbow.STL scale=1.0 1.0 1.0; visual mesh filename=package://coman_description/model/meshes/Elbow.STL scale=1.0 1.0 1.0
- link LFootmot: geometry collision mesh filename=package://coman_description/model/meshes/simple/Leg4.STL scale=0.03937 -0.03937 0.03937; visual mesh filename=package://coman_description/model/meshes/Leg4.STL scale=0.03937 -0.03937 0.03937
- link LForearm: geometry collision mesh filename=package://coman_description/model/meshes/simple/Forearm0.STL scale=1.0 1.0 1.0; visual mesh filename=package://coman_description/model/meshes/Forearm0.STL scale=0.1 0.1 0.1
- link LHipMot: geometry collision mesh filename=package://coman_description/model/meshes/simple/Leg0.STL scale=0.03937 -0.03937 0.03937; visual mesh filename=package://coman_description/model/meshes/Leg0.STL scale=0.03937 -0.03937 0.03937
- link LLowLeg: geometry collision mesh filename=package://coman_description/model/meshes/simple/Leg3.STL scale=0.03937 -0.03937 0.03937; visual mesh filename=package://coman_description/model/meshes/Leg3.STL scale=0.03937 -0.03937 0.03937
- link LShp: geometry collision mesh filename=package://coman_description/model/meshes/simple/Arm0.STL scale=0.03937 -0.03937 0.03937; visual mesh filename=package://coman_description/model/meshes/Arm0.STL scale=0.03937 -0.03937 0.03937
- link LShr: geometry collision mesh filename=package://coman_description/model/meshes/simple/Arm1.STL scale=0.03937 -0.03937 0.03937; visual mesh filename=package://coman_description/model/meshes/Arm1.STL scale=0.03937 -0.03937 0.03937
- link LShy: geometry collision mesh filename=package://coman_description/model/meshes/simple/Arm2.STL scale=0.03937 -0.03937 0.03937; visual mesh filename=package://coman_description/model/meshes/Arm2.STL scale=0.03937 -0.03937 0.03937
- link LSoftHand: geometry collision mesh filename=package://coman_description/model/meshes/simple/SoftHandOpe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 scale=-1E-3 1E-3 1E-3; visual mesh filename=package://coman_description/model/meshes/SoftHandOpen.STL scale=-0.1 0.1 0.1
- link LThighLowLeg: geometry collision mesh filename=package://coman_description/model/meshes/simple/Leg2.STL scale=0.03937 -0.03937 0.03937; visual mesh filename=package://coman_description/model/meshes/Leg2.STL scale=0.03937 -0.03937 0.03937
- link LThighUpLeg: geometry collision mesh filename=package://coman_description/model/meshes/simple/Leg1.STL scale=0.03937 -0.03937 0.03937; visual mesh filename=package://coman_description/model/meshes/Leg1.STL scale=0.03937 -0.03937 0.03937
- link LWrMot2: geometry collision mesh filename=package://coman_description/model/meshes/simple/Forearm1.STL scale=0.001 0.001 0.001; visual mesh filename=package://coman_description/model/meshes/Forearm1.STL scale=0.001 0.001 0.001
- link LWrMot3: geometry collision mesh filename=package://coman_description/model/meshes/simple/Forearm2.STL scale=0.001 0.001 0.001; visual mesh filename=package://coman_description/model/meshes/Forearm2.STL scale=0.001 0.001 0.001
- link RElb: geometry collision mesh filename=package://coman_description/model/meshes/simple/Elbow.STL scale=1.0 1.0 1.0; visual mesh filename=package://coman_description/model/meshes/Elbow.STL scale=1.0 1.0 1.0
- link RFootmot: geometry collision mesh filename=package://coman_description/model/meshes/simple/Leg4.STL scale=0.03937 0.03937 0.03937; visual mesh filename=package://coman_description/model/meshes/Leg4.STL scale=0.03937 0.03937 0.03937
- link RForearm: geometry collision mesh filename=package://coman_description/model/meshes/simple/Forearm0.STL scale=1.0 1.0 1.0; visual mesh filename=package://coman_description/model/meshes/Forearm0.STL scale=0.1 0.1 0.1
- link RHipMot: geometry collision mesh filename=package://coman_description/model/meshes/simple/Leg0.STL scale=0.03937 0.03937 0.03937; visual mesh filename=package://coman_description/model/meshes/Leg0.STL scale=0.03937 0.03937 0.03937
- link RLowLeg: geometry collision mesh filename=package://coman_description/model/meshes/simple/Leg3.STL scale=0.03937 0.03937 0.03937; visual mesh filename=package://coman_description/model/meshes/Leg3.STL scale=0.03937 0.03937 0.03937
- link RShp: geometry collision mesh filename=package://coman_description/model/meshes/simple/Arm0.STL scale=0.03937 0.03937 0.03937; visual mesh filename=package://coman_description/model/meshes/Arm0.STL scale=0.03937 0.03937 0.03937
- link RShr: geometry collision mesh filename=package://coman_description/model/meshes/simple/Arm1.STL scale=0.03937 0.03937 0.03937; visual mesh filename=package://coman_description/model/meshes/Arm1.STL scale=0.03937 0.03937 0.03937
- link RShy: geometry collision mesh filename=package://coman_description/model/meshes/simple/Arm2.STL scale=0.03937 0.03937 0.03937; visual mesh filename=package://coman_description/model/meshes/Arm2.STL scale=0.03937 0.03937 0.03937
- link RSoftHand: geometry collision mesh filename=package://coman_description/model/meshes/simple/SoftHandOpe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 scale=1E-3 1E-3 1E-3; visual mesh filename=package://coman_description/model/meshes/SoftHandOpen.STL scale=0.1 0.1 0.1
- link RThighLowLeg: geometry collision mesh filename=package://coman_description/model/meshes/simple/Leg2.STL scale=0.03937 0.03937 0.03937; visual mesh filename=package://coman_description/model/meshes/Leg2.STL scale=0.03937 0.03937 0.03937
- link RThighUpLeg: geometry collision mesh filename=package://coman_description/model/meshes/simple/Leg1.STL scale=0.03937 0.03937 0.03937; visual mesh filename=package://coman_description/model/meshes/Leg1.STL scale=0.03937 0.03937 0.03937
- link RWrMot2: geometry collision mesh filename=package://coman_description/model/meshes/simple/Forearm1.STL scale=0.001 0.001 0.001; visual mesh filename=package://coman_description/model/meshes/Forearm1.STL scale=0.001 0.001 0.001
- link RWrMot3: geometry collision mesh filename=package://coman_description/model/meshes/simple/Forearm2.STL scale=0.001 0.001 0.001; visual mesh filename=package://coman_description/model/meshes/Forearm2.STL scale=0.001 0.001 0.001
- link Waist: geometry collision mesh filename=package://coman_description/model/meshes/simple/Waist.STL scale=0.03937 0.03937 0.03937; visual mesh filename=package://coman_description/model/meshes/Waist.STL scale=0.03937 0.03937 0.03937
Joints:
- joint base_joint: origin xyz=0 0 0.55 rpy=0 0 0 -> xyz=0 0 0 rpy=0 0 0

Commit message: Fixed NaN issue

File: coman_description/model/model.urdf (robot description, URDF)
Before this commit: robot coman, 64 links, 63 joints
Joints:
- joint gaze_joint: origin xyz=0 0 0.1 rpy=0 0 0 -> xyz=0 0 0 rpy=0 0 0

Commit message: Sunglasses didnt work, implemented the camera instead.

File: coman_description/model/model.urdf (robot description, URDF)
Before this commit: robot coman, 64 links, 63 joints
Links:
- added link Xtion_cam_body, mass 0.2; visual box size=0.02 0.1 0.02
Joints:
- added joint Xtion_cam_joint: type fixed, parent torso, child Xtion_cam_body, origin xyz=0 0 0.1 rpy=0 0.05 0
- joint gaze_joint: origin xyz=0 0 0 rpy=0 0 0 -> xyz=0.015 0 0.022 rpy=0 0 0; parent torso -> Xtion_cam_body
